Commit message: 实现了在RVIZ2中实现基于位置控制的多项式步态规划

File: src/leg_module/leg_urdf/leg.urdf (robot description, URDF)
Before this commit: robot left_back_leg, 4 links, 3 joints
Links:
- removed link base_link
- added link link0; visual cylinder length=0.049 radius=0.04825
- added link world
Joints:
- added joint joint0: type fixed, parent world, child link0, origin xyz=0.115 -0.108 0.32 rpy=1.5708 1.5708 -1.5708
- joint joint1: parent base_link -> link0
